File: PCB/Uniform/Uniform.kicad_pcb (KiCad board)
At the start: 2 copper layers, 301.5 x 93.4 mm, 166 parts, among them U1 STM32L072KZT6

Commit message: v1 final gerber files submitted
Parts:
- removed the G*** at (55.7, 194.1)

Commit message: changed M3 mounting to M2.5 due to clearance issues
Parts:
- removed HOLE_M3 (x6): VAL**, keyboard_parts.pretty-master:HOLE_M3
- added REF**: MountingHole_2.7mm_M2.5, MountingHole:MountingHole_2.7mm_M2.5, F.Cu at (66.7, 181.0)
- added REF**: MountingHole_2.7mm_M2.5, MountingHole:MountingHole_2.7mm_M2.5, F.Cu at (314.3, 181.0)
- added REF**: MountingHole_2.7mm_M2.5, MountingHole:MountingHole_2.7mm_M2.5, F.Cu at (314.3, 123.8)
- added REF**: MountingHole_2.7mm_M2.5, MountingHole:MountingHole_2.7mm_M2.5, F.Cu at (66.7, 123.8)
- added REF**: MountingHole_2.7mm_M2.5, MountingHole:MountingHole_2.7mm_M2.5, F.Cu at (142.9, 165.0)
- added REF**: MountingHole_2.7mm_M2.5, MountingHole:MountingHole_2.7mm_M2.5, F.Cu at (238.1, 165.0)

Commit message: added mounting hole graphics
Parts:
- added G***: LOGO, Graphics:graphic_mounting_indicator, F.Cu at (42.8, 196.1)
- added G***: LOGO, Graphics:graphic_mounting_indicator, F.Cu at (238.1, 165.0)
- added G***: LOGO, Graphics:graphic_mounting_indicator, F.Cu at (66.7, 181.0)
- added G***: LOGO, Graphics:graphic_mounting_indicator, F.Cu at (314.3, 123.8)
- added G***: LOGO, Graphics:graphic_mounting_indicator, F.Cu at (66.7, 123.8)
- added G***: LOGO, Graphics:graphic_mounting_indicator, F.Cu at (314.3, 181.0)
- added G***: LOGO, Graphics:graphic_mounting_indicator, F.Cu at (142.9, 165.0)
- added G***: LOGO, Graphics:graphic_mounting_indicator, F.Cu at (42.8, 108.7)
- renumbered REF** to M1, REF** to M2, REF** to M3, REF** to M4, REF** to M5, REF** to M6
Changed lines of the file:
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@@
     )
     (pad_to_mask_clearance 0)
-    (grid_origin 142.875 164.30625)
+    (grid_origin 238.125 164.97525)
     (pcbplotparams
       (layerselection 0x00010fc_ffffffff)
@@
       (effects (font (size 1 1) (thickness 0.15)))
     )
-    (fp_text user "${REFERENCE}" (at 0.3 0) (layer "F.Fab")
+    (fp_text user "${REFERENCE}" (at 0.000001 3.15) (layer "F.SilkS")
       (effects (font (size 1 1) (thickness 0.15)))
     )
@@
       (effects (font (size 1 1) (thickness 0.15)))
     )
-    (fp_text user "${REFERENCE}" (at 0.3 0) (layer "F.Fab")
+    (fp_text user "${REFERENCE}" (at 3.75 0) (layer "F.SilkS")
       (effects (font (size 1 1) (thickness 0.15)))
     )
@@
     (tags "mounting hole 2.7mm no annular m2.5")
     (attr exclude_from_pos_files exclude_from_bom)
-    (fp_text reference "REF**" (at 0 -3.7) (layer "F.SilkS")
+    (fp_text reference "M3" (at -3.5 0) (layer "F.SilkS")
       (effects (font (size 1 1) (thickness 0.15)))
     )
@@
     (pad "" np_thru_hole circle (at 0 0) (size 2.7 2.7) (drill 2.7) (layers *.Cu *.Mask))
   )
+  (footprint "Graphics:graphic_mounting_indicator" (layer "F.Cu")
+    (at 42.775 196.1)
+    (attr board_only exclude_from_pos_files exclude_from_bom)
+    (fp_text reference "G***" (at 0 4) (layer "F.Fab")
+      (effects (font (size 1.524 1.524) (thickness 0.3)))
+    )
+    (fp_text value "LOGO" (at 0.75 0) (layer "F.SilkS") hide
+      (effects (font (size 1.524 1.524) (thickness 0.381)))
+    )
+    (fp_circle (center 0 0) (end 1.5 0) (layer "F.SilkS") (width 0.25) (fill none))
+    (fp_circle (center 0 0) (end 1.8 0) (layer "F.SilkS") (width 0.12) (fill none))
+  )
   (footprint "MountingHole:MountingHole_2.7mm_M2.5" (layer "F.Cu")
     (at 314.325 180.975)
@@
     (tags "mounting hole 2.7mm no annular m2.5")
     (attr exclude_from_pos_files exclude_from_bom)
-    (fp_text reference "REF**" (at 0 -3.7) (layer "F.SilkS")
+    (fp_text reference "M4" (at -3.4 0) (layer "F.SilkS")
       (effects (font (size 1 1) (thickness 0.15)))
     )
@@
     (pad "" np_thru_hole circle (at 0 0) (size 2.7 2.7) (drill 2.7) (layers *.Cu *.Mask))
   )
+  (footprint "Graphics:graphic_mounting_indicator" (layer "F.Cu")
+    (at 238.125 164.97525)
+    (attr board_only exclude_from_pos_files exclude_from_bom)
+    (fp_text reference "G***" (at 0 4) (layer "F.Fab")
+      (effects (font (size 1.524 1.524) (thickness 0.3)))
+    )
+    (fp_text value "LOGO" (at 0.75 0) (layer "F.SilkS") hide
+      (effects (font (size 1.524 1.524) (thickness 0.381)))
+    )
+    (fp_circle (center 0 0) (end 1.5 0) (layer "F.SilkS") (width 0.25) (fill none))
+    (fp_circle (center 0 0) (end 1.8 0) (layer "F.SilkS") (width 0.12) (fill none))
+  )
   (footprint "Graphics:graphic_logo" (layer "F.Cu")
     (at 48.6375 156.7)
@@
     (tags "mounting hole 2.7mm no annular m2.5")
     (attr exclude_from_pos_files exclude_from_bom)
-    (fp_text reference "REF**" (at 0 -3.7) (layer "F.SilkS")
+    (fp_text reference "M2" (at -3.4 0) (layer "F.SilkS")
       (effects (font (size 1 1) (thickness 0.15)))
     )
@@
     (pad "" np_thru_hole circle (at 0 0) (size 2.7 2.7) (drill 2.7) (layers *.Cu *.Mask))
   )
+  (footprint "Graphics:graphic_mounting_indicator" (layer "F.Cu")
+    (at 66.675 180.975)
+    (attr board_only exclude_from_pos_files exclude_from_bom)
+    (fp_text reference "G***" (at 0 4) (layer "F.Fab")
+      (effects (font (size 1.524 1.524) (thickness 0.3)))
+    )
+    (fp_text value "LOGO" (at 0.75 0) (layer "F.SilkS") hide
+      (effects (font (size 1.524 1.524) (thickness 0.381)))
+    )
+    (fp_circle (center 0 0) (end 1.5 0) (layer "F.SilkS") (width 0.25) (fill none))
+    (fp_circle (center 0 0) (end 1.8 0) (layer "F.SilkS") (width 0.12) (fill none))
+  )
   (footprint "MountingHole:MountingHole_2.7mm_M2.5" (layer "F.Cu")
     (at 66.675 123.825)
@@
     (tags "mounting hole 2.7mm no annular m2.5")
     (attr exclude_from_pos_files exclude_from_bom)
-    (fp_text reference "REF**" (at 0 -3.7) (layer "F.SilkS")
+    (fp_text reference "M1" (at -3.5 0) (layer "F.SilkS")
       (effects (font (size 1 1) (thickness 0.15)))
     )
@@
     (tags "mounting hole 2.7mm no annular m2.5")
     (attr exclude_from_pos_files exclude_from_bom)
-    (fp_text reference "REF**" (at 0 -3.7) (layer "F.SilkS")
+    (fp_text reference "M5" (at 0 -3) (layer "F.SilkS")
       (effects (font (size 1 1) (thickness 0.15)))
     )
@@
     (pad "" np_thru_hole circle (at 0 0) (size 2.7 2.7) (drill 2.7) (layers *.Cu *.Mask))
   )
+  (footprint "Graphics:graphic_mounting_indicator" (layer "F.Cu")
+    (at 314.325 123.825)
+    (attr board_only exclude_from_pos_files exclude_from_bom)
+    (fp_text reference "G***" (at 0 4) (layer "F.Fab")
+      (effects (font (size 1.524 1.524) (thickness 0.3)))
+    )
+    (fp_text value "LOGO" (at 0.75 0) (layer "F.SilkS") hide
+      (effects (font (size 1.524 1.524) (thickness 0.381)))
+    )
+    (fp_circle (center 0 0) (end 1.8 0) (layer "F.SilkS") (width 0.12) (fill none))
+    (fp_circle (center 0 0) (end 1.5 0) (layer "F.SilkS") (width 0.25) (fill none))
+  )
   (footprint "MountingHole:MountingHole_2.7mm_M2.5" (layer "F.Cu")
     (at 238.125 164.97525)
@@
     (tags "mounting hole 2.7mm no annular m2.5")
     (attr exclude_from_pos_files exclude_from_bom)
-    (fp_text reference "REF**" (at 0 -3.7) (layer "F.SilkS")
+    (fp_text reference "M6" (at 0 -3) (layer "F.SilkS")
       (effects (font (size 1 1) (thickness 0.15)))
     )
@@
     (pad "" np_thru_hole circle (at 0 0) (size 2.7 2.7) (drill 2.7) (layers *.Cu *.Mask))
   )
+  (footprint "Graphics:graphic_mounting_indicator" (layer "F.Cu")
+    (at 66.675 123.825)
+    (attr board_only exclude_from_pos_files exclude_from_bom)
+    (fp_text reference "G***" (at 0 4) (layer "F.Fab")
+      (effects (font (size 1.524 1.524) (thickness 0.3)))
+    )
+    (fp_text value "LOGO" (at 0.75 0) (layer "F.SilkS") hide
+      (effects (font (size 1.524 1.524) (thickness 0.381)))
+    )
+    (fp_circle (center 0 0) (end 1.8 0) (layer "F.SilkS") (width 0.12) (fill none))
+    (fp_circle (center 0 0) (end 1.5 0) (layer "F.SilkS") (width 0.25) (fill none))
+  )
+  (footprint "Graphics:graphic_mounting_indicator" (layer "F.Cu")
+    (at 314.325 180.975)
+    (attr board_only exclude_from_pos_files exclude_from_bom)
+    (fp_text reference "G***" (at 0 4) (layer "F.Fab")
+      (effects (font (size 1.524 1.524) (thickness 0.3)))
+    )
+    (fp_text value "LOGO" (at 0.75 0) (layer "F.SilkS") hide
+      (effects (font (size 1.524 1.524) (thickness 0.381)))
+    )
+    (fp_circle (center 0 0) (end 1.8 0) (layer "F.SilkS") (width 0.12) (fill none))
+    (fp_circle (center 0 0) (end 1.5 0) (layer "F.SilkS") (width 0.25) (fill none))
+  )
+  (footprint "Graphics:graphic_mounting_indicator" (layer "F.Cu")
+    (at 142.875 164.97525)
+    (attr board_only exclude_from_pos_files exclude_from_bom)
+    (fp_text reference "G***" (at 0 4) (layer "F.Fab")
+      (effects (font (size 1.524 1.524) (thickness 0.3)))
+    )
+    (fp_text value "LOGO" (at 0.75 0) (layer "F.SilkS") hide
+      (effects (font (size 1.524 1.524) (thickness 0.381)))
+    )
+    (fp_circle (center 0 0) (end 1.8 0) (layer "F.SilkS") (width 0.12) (fill none))
+    (fp_circle (center 0 0) (end 1.5 0) (layer "F.SilkS") (width 0.25) (fill none))
+  )
+  (footprint "Graphics:graphic_mounting_indicator" (layer "F.Cu")
+    (at 42.775001 108.700001)
+    (attr board_only exclude_from_pos_files exclude_from_bom)
+    (fp_text reference "G***" (at 0 4) (layer "F.Fab")
+      (effects (font (size 1.524 1.524) (thickness 0.3)))
+    )
+    (fp_text value "LOGO" (at 0.75 0) (layer "F.SilkS") hide
+      (effects (font (size 1.524 1.524) (thickness 0.381)))
+    )
+    (fp_circle (center 0 0) (end 1.5 0) (layer "F.SilkS") (width 0.25) (fill none))
+    (fp_circle (center 0 0) (end 1.8 0) (layer "F.SilkS") (width 0.12) (fill none))
+  )
   (footprint "USB4085-GF-A_REVA4:GCT_USB4085-GF-A_REVA4" (layer "B.Cu")

Commit message: Moved mount holes so the drill points in the plate won't collide with switch clip-in points
Parts:
- added G***: LOGO, Graphics:graphic_mounting_indicator, F.Cu at (219.1, 123.8)
- added G***: LOGO, Graphics:graphic_mounting_indicator, F.Cu at (161.9, 123.8)
- added M5: MountingHole_2.7mm_M2.5, MountingHole:MountingHole_2.7mm_M2.5, F.Cu at (219.1, 123.8)
- added M5: MountingHole_2.7mm_M2.5, MountingHole:MountingHole_2.7mm_M2.5, F.Cu at (161.9, 123.8)
- moved G*** 38.1 mm to (104.8, 181.0)
- moved G*** 38.1 mm to (104.8, 123.8)
- moved M1 38.1 mm to (104.8, 123.8)
- moved M3 38.1 mm to (104.8, 181.0)
- moved G*** 38.1 mm to (276.2, 123.8)
- moved G*** 38.1 mm to (276.2, 181.0)
- moved M2 38.1 mm to (276.2, 123.8)
- moved M4 38.1 mm to (276.2, 181.0)
- moved G*** 24.9 mm to (219.1, 181.0)
- moved G*** 24.9 mm to (161.9, 181.0)
- moved M5 24.9 mm to (161.9, 181.0)
- moved M6 24.9 mm to (219.1, 181.0)
- moved D_3_0 19.2 mm to (81.0, 171.4)
- moved D_0_0 19.2 mm to (81.0, 114.3)
- moved D_1_0 19.2 mm to (81.0, 133.3)
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Routing:
- net GND: track 197.8 -> 206.5 mm
- net Net-(D_2_0-Pad2): track 6.04 -> 14.0 mm
- net Net-(D_0_0-Pad2): track 6.04 -> 14.0 mm
- net Net-(D_4_0-Pad2): track 6.04 -> 14.0 mm
- net Net-(D_3_0-Pad2): track 6.04 -> 14.0 mm
- net Net-(D_1_0-Pad2): track 6.04 -> 14.0 mm
- net R0: track 325.8 -> 328.3 mm, vias 1 -> 2
- net R4: track 295.0 -> 292.7 mm
- net R1: track 305.3 -> 306.9 mm, vias 1 -> 2
- net R2: track 290.3 -> 291.3 mm, vias 1 -> 2
- net R3: track 276.5 -> 275.6 mm

Commit message: Added Neopixel status LED, moved mount holes, and re-routed traces to fit new status led type
Parts:
- added G***: LOGO, Graphics:graphic_mounting_indicator, F.Cu at (304.8, 123.8)
- added G***: LOGO, Graphics:graphic_logo, B.Cu at (52.4, 162.3)
- added G***: LOGO, Graphics:graphic_designed-by-with-year, B.Cu at (52.7, 166.3)
- added G***: LOGO, Graphics:graphic_mounting_indicator, F.Cu at (76.2, 123.8)
- added G***: LOGO, Graphics:graphic_mounting_indicator, F.Cu at (304.8, 181.0)
- added G***: LOGO, Graphics:graphic_mounting_indicator, F.Cu at (76.2, 181.0)
- added M1: MountingHole_2.7mm_M2.5, MountingHole:MountingHole_2.7mm_M2.5, F.Cu at (76.2, 123.8)
- added M12: MountingHole_2.7mm_M2.5, MountingHole:MountingHole_2.7mm_M2.5, F.Cu at (304.8, 181.0)
- added M6: MountingHole_2.7mm_M2.5, MountingHole:MountingHole_2.7mm_M2.5, F.Cu at (304.8, 123.8)
- added M7: MountingHole_2.7mm_M2.5, MountingHole:MountingHole_2.7mm_M2.5, F.Cu at (76.2, 181.0)
- LED1: value LED -> NeoPixel_THT; footprint LED_THT:LED_D3.0mm_Clear -> LED_THT:LED_D5.0mm-4_RGB
- moved LED1 0.65 mm to (50.4, 111.8)
- renumbered M6 to M10, M4 to M11, M1 to M2, M5 to M3, M5 to M4, M2 to M5, M3 to M8, M5 to M9, SWD to SWD1, V_REG to VREG1
Connections:
- LED1 pad 1: GND -> unconnected-(LED1-Pad1)
- LED1 pad 2: Net-(LED1-Pad2) -> GND
- R6 pad 2: Net-(LED1-Pad2) -> Net-(LED1-Pad4)
Routing:
- net Net-(LED1-Pad2): track 43.0 -> 0.00 mm
- net Net-(LED1-Pad4): track 0.00 -> 42.7 mm
- net +5V: track 40.0 -> 49.7 mm
- net GND: track 206.5 -> 210.1 mm
- net Net-(R1-Pad2): track 16.4 -> 18.3 mm
