File: PCB/Uniform_Board/Uniform_Board.kicad_pcb (KiCad board)
At the start: 2 copper layers, 301.5 x 93.4 mm, 186 parts, among them M1 MountingHole_2.7mm_M2.5, M10 MountingHole_2.7mm_M2.5, M2 MountingHole_2.7mm_M2.5, M3 MountingHole_2.7mm_M2.5, M4 MountingHole_2.7mm_M2.5, M5 MountingHole_2.7mm_M2.5, M6 MountingHole_2.7mm_M2.5, M7 MountingHole_2.7mm_M2.5, M8 MountingHole_2.7mm_M2.5, M9 MountingHole_2.7mm_M2.5, U1 STM32L072KZT6, U2 SN74AHCT1G125DBVR

Commit message: board USBC and power routed to PCIE, pre row/column routing
Parts:
- removed C1, C2: 10uf, ul_FG16X7R1E106KRT06:FG16X7R1E106KRT06
- removed C3, C4, C5: 0.1uf, Resistor_THT:R_Axial_DIN0207_L6.3mm_D2.5mm_P7.62mm_Horizontal
- removed C6: 1uf, RDER71H105K2M1H03A:CAP_RDER71H105K2M1H03A
- removed the G*** at (48.6, 156.7)
- removed L1, L2, L3: NeoPixel_THT, Neopixel:LED_D5.0mm-4_RGB
- removed L4: Conn_01x03, Connector_PinHeader_2.54mm:PinHeader_1x03_P2.54mm_Vertical
- removed R3, R4: 10k, Resistor_THT:R_Axial_DIN0204_L3.6mm_D1.6mm_P7.62mm_Horizontal
- removed R5: R, Resistor_THT:R_Axial_DIN0309_L9.0mm_D3.2mm_P12.70mm_Horizontal
- removed R6: 330, Resistor_THT:R_Axial_DIN0309_L9.0mm_D3.2mm_P12.70mm_Horizontal
- removed S1, S2: OS102011MS2QN1, OS102011MS2QN1:SW_OS102011MS2QN1
- removed SWD1: 826629-5, 826629-5:TE_826629-5
- removed U1: STM32L072KZT6, STM32L072KZT6:QFP80P900X900X160-32N
- removed U2: SN74AHCT1G125DBVR, SN74AHCT1G125DBVR:SOT95P280X145-5N
- removed VREG1: TLV1117-33, TLV1117-33IDCY:SOT230P700X180-4N
- added J1: PCIE_x1_SAMTEC_PCIE-036-02-F-D-TH, Uniform:SAMTEC_PCIE-036-02-F-D-TH, F.Cu at (49.0, 128.4)
- D_0_0, D_0_1, D_0_10, D_0_11, D_0_12, D_0_13, D_0_2, D_0_3, D_0_4, D_0_5, D_0_6, D_0_7, D_0_8, D_0_9, D_1_0, D_1_1, D_1_10, D_1_11, D_1_12, D_1_13, D_1_2, D_1_3, D_1_4, D_1_5, D_1_6, D_1_7, D_1_8, D_1_9, D_2_0, D_2_1, D_2_10, D_2_11, D_2_12, D_2_13, D_2_2, D_2_3, D_2_4, D_2_5, D_2_6, D_2_7, D_2_8, D_2_9, D_3_0, D_3_1, D_3_10, D_3_11, D_3_12, D_3_13, D_3_2, D_3_3, D_3_4, D_3_5, D_3_6, D_3_7, D_3_8, D_3_9, D_4_0, D_4_1, D_4_10, D_4_11, D_4_12, D_4_13, D_4_2, D_4_4, D_4_5, D_4_6, D_4_8, D_4_9: footprint 1N4148:DIOAD829W49L456D191 -> Uniform:Diode_DIOAD829W49L456D191
- R1, R2: footprint Resistor_THT:R_Axial_DIN0204_L3.6mm_D1.6mm_P7.62mm_Horizontal -> Resistor_SMD:R_0603_1608Metric_Pad0.98x0.95mm_HandSolder
- USBC1: footprint USB4085-GF-A_REVA4:GCT_USB4085-GF-A_REVA4 -> Uniform:USBC_USB4085-GF-A
- moved R1 17.2 mm to (48.5, 108.5), turned to 0 degrees
- moved R2 14.2 mm to (48.5, 110.7), turned to 0 degrees
Routing:
- net GND: track 191.9 -> 46.4 mm, vias 1 -> 0
- net +3V3: track 114.3 -> 0.00 mm, vias 3 -> 0
- net R0: track 327.5 -> 257.0 mm, vias 2 -> 0
- net RESET: track 61.9 -> 0.00 mm, vias 1 -> 0
- net +5V: track 72.8 -> 22.8 mm, vias 1 -> 0
- net D_N: track 68.6 -> 22.2 mm
- net D_P: track 69.3 -> 24.2 mm
- net C13: track 397.4 -> 353.4 mm, vias 2 -> 0
- net STATUS_LED_DATA: track 42.8 -> 0.00 mm
- net C12: track 366.4 -> 332.1 mm
- net C11: track 340.2 -> 307.0 mm
- net C10: track 315.8 -> 283.6 mm
- net LED_DATA: track 31.2 -> 0.00 mm
- net R2: track 291.3 -> 262.9 mm, vias 2 -> 0
- net R4: track 293.7 -> 265.7 mm
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Other:
- board text removed: "BOOT->"
- board text removed: "RESET->"

Commit message: started board routing; first attempt
Connections:
- J1 pad A1: C11 -> C2
- J1 pad A2: C12 -> C1
- J1 pad A3: C13 -> C0
- J1 pad B1: C10 -> C3
- J1 pad B10: C1 -> C12
- J1 pad B11: C0 -> C13
- J1 pad B2: C8 -> C4
- J1 pad B3: C9 -> C5
- J1 pad B4: C7 -> C6
- J1 pad B5: C6 -> C7
- J1 pad B6: C5 -> C8
- J1 pad B7: C4 -> C9
- J1 pad B8: C3 -> C10
- J1 pad B9: C2 -> C11
Routing:
- net R4: track 265.7 -> 340.8 mm, vias 0 -> 1
- net R3: track 267.2 -> 324.1 mm, vias 0 -> 1
- net C0: track 88.2 -> 132.8 mm
- net R2: track 262.9 -> 303.4 mm, vias 0 -> 1
- net C1: track 112.4 -> 152.1 mm
- net C2: track 131.8 -> 168.9 mm
- net C3: track 139.0 -> 167.6 mm
- net C7: track 218.7 -> 246.9 mm
- net C5: track 197.9 -> 225.5 mm
- net C9: track 277.5 -> 304.9 mm
- net C6: track 219.8 -> 247.0 mm
- net C4: track 179.9 -> 206.1 mm
- net C8: track 257.6 -> 283.5 mm
- net C11: track 307.0 -> 332.6 mm
- net C13: track 353.4 -> 378.6 mm
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
Commit message: rework routing on board, cleaner!
Routing:
- net C6: track 247.0 -> 225.7 mm
- net C7: track 246.9 -> 226.2 mm
- net C8: track 283.5 -> 262.7 mm
- net C9: track 304.9 -> 284.1 mm
- net C5: track 225.5 -> 206.3 mm
- net C3: track 167.6 -> 148.3 mm
- net C4: track 206.1 -> 186.8 mm
- net C0: track 132.8 -> 114.5 mm
- net C1: track 152.1 -> 134.0 mm
- net C2: track 168.9 -> 150.8 mm
- net C10: track 307.6 -> 301.6 mm
- net C11: track 332.6 -> 327.0 mm
- net C12: track 355.3 -> 350.2 mm
- net C13: track 378.6 -> 373.5 mm

Commit message: finished uniform board routing
Routing:
- net R1: track 283.9 -> 278.8 mm
- net R4: track 340.8 -> 336.3 mm
- net R3: track 324.1 -> 320.0 mm
- net R2: track 303.4 -> 299.8 mm
- net C13: track 373.5 -> 372.5 mm
- net C12: track 350.2 -> 349.2 mm
- net C11: track 327.0 -> 326.0 mm
- net C10: track 301.6 -> 300.6 mm
- net C9: track 284.1 -> 283.1 mm
- net C8: track 262.7 -> 261.6 mm
- net C4: track 186.8 -> 185.8 mm
- net C7: track 226.2 -> 225.1 mm
- net C3: track 148.3 -> 147.3 mm
- net C6: track 225.7 -> 224.7 mm
- net C5: track 206.3 -> 205.3 mm
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
Commit message: fixed some minor routing issues on uniform board, removed silkscreen diode ref text
Parts:
- moved R2 0.92 mm to (49.1, 110.0)
- moved R1 0.63 mm to (49.1, 108.3)
Routing:
- net GND: track 46.4 -> 53.0 mm
- net Net-(R1-Pad2): track 9.54 -> 9.02 mm

Commit message: finishing touches on silkscreen graphics for board
Parts:
- added G***: LOGO, Graphics:graphic_logo, F.Cu at (48.9, 143.0)
- moved G*** 30.4 mm to (56.8, 196.5)
- moved G*** 28.8 mm to (57.3, 190.7)
Other:
- board text added: "2024"
- board text added: "v2.00"

Commit message: PCIE Edge Connector footprint dimmensions and edge cuts done
Parts:
- moved J1 1.34 mm to (47.7, 128.4), turned to 90 degrees
- moved G*** 1.20 mm to (47.7, 143.0)
Connections:
- J1 pad A1: C2 -> +5V
- J1 pad A10: unconnected-(J1-PadA10) -> C5
- J1 pad A11: unconnected-(J1-PadA11) -> C4
- J1 pad A12: unconnected-(J1-PadA12) -> C3
- J1 pad A13: unconnected-(J1-PadA13) -> C2
- J1 pad A14: D_P -> C1
- J1 pad A15: unconnected-(J1-PadA15) -> C0
- J1 pad A16: D_N -> unconnected-(J1-PadA16)
- J1 pad A17: GND -> unconnected-(J1-PadA17)
- J1 pad A18: +5V -> unconnected-(J1-PadA18)
- J1 pad A2: C1 -> C13
- J1 pad A3: C0 -> C12
- J1 pad A4: unconnected-(J1-PadA4) -> C11
- J1 pad A5: unconnected-(J1-PadA5) -> C10
- J1 pad A6: unconnected-(J1-PadA6) -> C9
- J1 pad A7: unconnected-(J1-PadA7) -> C8
- J1 pad A8: unconnected-(J1-PadA8) -> C7
- J1 pad A9: unconnected-(J1-PadA9) -> C6
- J1 pad B1: C3 -> GND
- J1 pad B10: C12 -> unconnected-(J1-PadB10)
- J1 pad B11: C13 -> unconnected-(J1-PadB11)
- J1 pad B12: R4 -> unconnected-(J1-PadB12)
- J1 pad B13: R3 -> unconnected-(J1-PadB13)
- J1 pad B14: R2 -> unconnected-(J1-PadB14)
- J1 pad B15: R1 -> unconnected-(J1-PadB15)
- J1 pad B16: R0 -> unconnected-(J1-PadB16)
- J1 pad B17: GND -> unconnected-(J1-PadB17)
- J1 pad B2: C4 -> D_P
- J1 pad B3: C5 -> D_N
- J1 pad B4: C6 -> R4
- J1 pad B5: C7 -> R3
- J1 pad B6: C8 -> R2
- J1 pad B7: C9 -> R1
- J1 pad B8: C10 -> R0
- J1 pad B9: C11 -> unconnected-(J1-PadB9)
Routing:
- net R4: track 336.3 -> 254.2 mm
- net R3: track 320.0 -> 254.2 mm
- net R2: track 299.8 -> 254.2 mm
- net R1: track 278.8 -> 257.7 mm
- net R0: track 268.4 -> 255.5 mm, vias 0 -> 1
- net C8: track 261.6 -> 272.0 mm
- net C4: track 185.8 -> 196.1 mm
- net C10: track 300.6 -> 310.9 mm
- net C6: track 224.7 -> 235.0 mm
- net C12: track 349.2 -> 359.5 mm
- net GND: track 53.0 -> 45.8 mm
- net C11: track 326.0 -> 332.3 mm
- net C7: track 225.1 -> 231.5 mm
- net C9: track 283.1 -> 289.4 mm
- net C5: track 205.3 -> 211.6 mm
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
Commit message: improved trace origins on PCIE port/edge. Board rerouting done. Module rerouting in progress
Connections:
- J1 pad A1: +5V -> C13
- J1 pad A10: C5 -> C4
- J1 pad A11: C4 -> C3
- J1 pad A12: C3 -> C2
- J1 pad A13: C2 -> C1
- J1 pad A14: C1 -> C0
- J1 pad A15: C0 -> unconnected-(J1-PadA15)
- J1 pad A18: unconnected-(J1-PadA18) -> +5V
- J1 pad A2: C13 -> C12
- J1 pad A3: C12 -> C11
- J1 pad A4: C11 -> C10
- J1 pad A5: C10 -> C9
- J1 pad A6: C9 -> C8
- J1 pad A7: C8 -> C7
- J1 pad A8: C7 -> C6
- J1 pad A9: C6 -> C5
- J1 pad B1: GND -> D_P
- J1 pad B18: unconnected-(J1-PadB18) -> GND
- J1 pad B2: D_P -> D_N
- J1 pad B3: D_N -> R4
- J1 pad B4: R4 -> R3
- J1 pad B5: R3 -> R2
- J1 pad B6: R2 -> R1
- J1 pad B7: R1 -> R0
- J1 pad B8: R0 -> unconnected-(J1-PadB8)
Routing:
- net R4: track 254.2 -> 360.4 mm
- net R3: track 254.2 -> 337.5 mm
- net R0: track 255.5 -> 322.7 mm
- net R2: track 254.2 -> 319.4 mm
- net R1: track 257.7 -> 303.7 mm
- net +5V: track 17.2 -> 35.4 mm
- net GND: track 45.8 -> 62.2 mm
- net C3: track 151.2 -> 156.3 mm
- net C13: track 378.8 -> 381.5 mm
- net C5: track 211.6 -> 214.3 mm
- net C9: track 289.4 -> 292.1 mm
- net C7: track 231.5 -> 234.2 mm
- net C11: track 332.3 -> 335.0 mm
- net D_P: track 18.5 -> 15.8 mm
- net C1: track 131.3 -> 133.8 mm
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